File: hw4/me433.brd (EAGLE design)
At the start: 160 x 100 mm, 27 parts

Commit message: made board layout
Parts:
- moved U$7 106.9 mm to (44.7, 5.84)
- moved U$12 100.6 mm to (47.0, 36.8), turned to 270 degrees
- moved U$10 96.6 mm to (36.8, 16.5)
- moved R3 95.9 mm to (44.5, 39.4), turned to 180 degrees
- moved U$2 88.8 mm to (27.1, 4.57), turned to 270 degrees
- moved U$11 85.9 mm to (36.8, 14.0)
- moved U$8 84.8 mm to (45.5, 46.5), turned to 180 degrees
- moved LED1 82.3 mm to (39.4, 45.7), turned to 90 degrees
- moved C3 76.7 mm to (31.8, 20.3), turned to 270 degrees
- moved U$16 76.4 mm to (2.54, 11.2)
- moved R1 74.2 mm to (43.2, 41.9)
- moved U$13 67.8 mm to (47.0, 24.1), turned to 270 degrees
- moved C1 67.0 mm to (33.0, 40.6), turned to 270 degrees
- moved U$18 62.0 mm to (8.89, 11.4)
- moved C2 60.3 mm to (18.5, 12.6), turned to 90 degrees
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Connections:
- removed net N$3: U$16.P$1
- removed net N$6: U$17.P$1
- net +3V3: now also U$16.P$1
- net GND: now also U$17.P$1
Routing:
- net +3V3: track 0.00 -> 167.1 mm, vias 0 -> 2
- net VIN: track 0.00 -> 66.9 mm, vias 0 -> 3
- net MCLR: track 0.00 -> 41.8 mm
- net B4: track 0.00 -> 39.6 mm, vias 0 -> 1
- net A4: track 0.00 -> 38.1 mm, vias 0 -> 2
- net B6: track 0.00 -> 34.2 mm, vias 0 -> 1
- net B5: track 0.00 -> 29.4 mm, vias 0 -> 2
- net U1TX: track 0.00 -> 29.0 mm
- net U1RX: track 0.00 -> 28.6 mm, vias 0 -> 1
- net B7: track 0.00 -> 25.2 mm, vias 0 -> 2
- net A3: track 0.00 -> 23.4 mm
- net +5V: track 0.00 -> 20.5 mm
- net PGC: track 0.00 -> 20.4 mm
- net B2: track 0.00 -> 20.1 mm
- net A1: track 0.00 -> 20.1 mm
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- added copper zone on layer 16, net GND
Other:
- board size 160 x 100 mm -> 50 x 50 mm
- board text added: "+"
- board text added: "+3V3"
- board text added: "3V3"
- board text added: "A0"
- board text added: "A1"
- board text added: "A3"
- board text added: "ABLAZA, ME433 2022"
- board text added: "B10"
- board text added: "B11"
- board text added: "B12"
- board text added: "B13"
- board text added: "B14"
- board text added: "B15"
- board text added: "B2"
- board text added: "B5"
- board text added: "B6"
- board text added: "B7"
- board text added: "GND"
- board text added: "VIN"
