File: hw4/me433.sch (EAGLE design)
At the start: 27 parts

Commit message: made board layout
Connections:
- removed net N$3: U$16.P$1
- removed net N$6: U$17.P$1
- net +3V3: now also U$16.P$1
- net GND: now also U$17.P$1
Other:
- moved on the sheet: U$15
Changed lines of the file:
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@@
 <part name="R3" library="me433" deviceset="R-US_" device="0207/7" package3d_urn="urn:adsk.eagle:package:23493/2" value="10k"/>
 <part name="R4" library="me433" deviceset="R-US_" device="0207/7" package3d_urn="urn:adsk.eagle:package:23493/2" value="10k"/>
-<part name="GND1" library="me433" deviceset="GND" device=""/>
-<part name="+3V1" library="me433" deviceset="+3V3" device=""/>
-<part name="P+1" library="me433" deviceset="+5V" device=""/>
 <part name="GND2" library="me433" deviceset="GND" device=""/>
 <part name="+3V2" library="me433" deviceset="+3V3" device=""/>
@@
 <part name="U$17" library="me433" deviceset="ONE" device=""/>
 <part name="U$18" library="me433" deviceset="ONE" device=""/>
-<part name="+3V12" library="me433" deviceset="+3V3" device=""/>
 <part name="GND18" library="me433" deviceset="GND" device=""/>
+<part name="+3V1" library="me433" deviceset="+3V3" device=""/>
 </parts>
 <sheets>
@@
 <attribute name="VALUE" x="219.202" y="118.11" size="1.778" layer="96" rot="R90"/>
 </instance>
-<instance part="GND1" gate="1" x="-5.08" y="63.5" smashed="yes">
-<attribute name="VALUE" x="-7.62" y="60.96" size="1.778" layer="96"/>
-</instance>
-<instance part="+3V1" gate="G$1" x="5.08" y="66.04" smashed="yes">
-<attribute name="VALUE" x="2.54" y="60.96" size="1.778" layer="96" rot="R90"/>
-</instance>
-<instance part="P+1" gate="1" x="12.7" y="66.04" smashed="yes">
-<attribute name="VALUE" x="10.16" y="60.96" size="1.778" layer="96" rot="R90"/>
-</instance>
 <instance part="GND2" gate="1" x="15.24" y="119.38" smashed="yes">
 <attribute name="VALUE" x="12.7" y="116.84" size="1.778" layer="96"/>
@@
 <attribute name="VALUE" x="223.52" y="12.7" size="1.27" layer="94"/>
 </instance>
-<instance part="U$15" gate="G$1" x="215.9" y="-20.32" smashed="yes">
-<attribute name="NAME" x="223.52" y="-17.78" size="1.27" layer="94"/>
-<attribute name="VALUE" x="223.52" y="-20.32" size="1.27" layer="94"/>
+<instance part="U$15" gate="G$1" x="218.44" y="-20.32" smashed="yes">
+<attribute name="NAME" x="226.06" y="-17.78" size="1.27" layer="94"/>
+<attribute name="VALUE" x="226.06" y="-20.32" size="1.27" layer="94"/>
 </instance>
 <instance part="+3V10" gate="G$1" x="195.58" y="40.64" smashed="yes">
@@
 <attribute name="VALUE" x="-48.26" y="10.16" size="1.27" layer="94"/>
 </instance>
-<instance part="+3V12" gate="G$1" x="-58.42" y="43.18" smashed="yes">
-<attribute name="VALUE" x="-60.96" y="38.1" size="1.778" layer="96" rot="R90"/>
-</instance>
 <instance part="GND18" gate="1" x="-55.88" y="25.4" smashed="yes">
 <attribute name="VALUE" x="-58.42" y="22.86" size="1.778" layer="96"/>
+</instance>
+<instance part="+3V1" gate="G$1" x="-58.42" y="43.18" smashed="yes">
+<attribute name="VALUE" x="-60.96" y="38.1" size="1.778" layer="96" rot="R90"/>
 </instance>
 </instances>
@@
 <junction x="198.12" y="2.54"/>
 <pinref part="GND17" gate="1" pin="GND"/>
+</segment>
+<segment>
+<pinref part="U$17" gate="G$1" pin="P$1"/>
+<wire x1="-50.8" y1="27.94" x2="-55.88" y2="27.94" width="0.1524" layer="91"/>
+<pinref part="GND18" gate="1" pin="GND"/>
+<label x="-55.88" y="27.94" size="1.778" layer="95"/>
 </segment>
 </net>
@@
 <pinref part="+3V11" gate="G$1" pin="+3V3"/>
 </segment>
+<segment>
+<pinref part="U$16" gate="G$1" pin="P$1"/>
+<wire x1="-50.8" y1="40.64" x2="-58.42" y2="40.64" width="0.1524" layer="91"/>
+<pinref part="+3V1" gate="G$1" pin="+3V3"/>
+</segment>
 </net>
 <net name="+5V" class="0">
@@
 <segment>
 <pinref part="U$15" gate="G$1" pin="P$1"/>
-<wire x1="210.82" y1="-10.16" x2="203.2" y2="-10.16" width="0.1524" layer="91"/>
+<wire x1="213.36" y1="-10.16" x2="203.2" y2="-10.16" width="0.1524" layer="91"/>
 <label x="205.74" y="-10.16" size="1.778" layer="95"/>
 </segment>
@@
 <segment>
 <pinref part="U$15" gate="G$1" pin="P$2"/>
-<wire x1="210.82" y1="-15.24" x2="203.2" y2="-15.24" width="0.1524" layer="91"/>
+<wire x1="213.36" y1="-15.24" x2="203.2" y2="-15.24" width="0.1524" layer="91"/>
 <label x="205.74" y="-15.24" size="1.778" layer="95"/>
 </segment>
@@
 <segment>
 <pinref part="U$15" gate="G$1" pin="P$3"/>
-<wire x1="210.82" y1="-20.32" x2="203.2" y2="-20.32" width="0.1524" layer="91"/>
+<wire x1="213.36" y1="-20.32" x2="203.2" y2="-20.32" width="0.1524" layer="91"/>
 <label x="205.74" y="-20.32" size="1.778" layer="95"/>
 </segment>
@@
 <segment>
 <pinref part="U$15" gate="G$1" pin="P$4"/>
-<wire x1="210.82" y1="-25.4" x2="200.66" y2="-25.4" width="0.1524" layer="91"/>
+<wire x1="213.36" y1="-25.4" x2="200.66" y2="-25.4" width="0.1524" layer="91"/>
 <label x="203.2" y="-25.4" size="1.778" layer="95"/>
 </segment>
@@
 <segment>
 <pinref part="U$15" gate="G$1" pin="P$5"/>
-<wire x1="210.82" y1="-30.48" x2="203.2" y2="-30.48" width="0.1524" layer="91"/>
+<wire x1="213.36" y1="-30.48" x2="203.2" y2="-30.48" width="0.1524" layer="91"/>
 <label x="205.74" y="-30.48" size="1.778" layer="95"/>
 </segment>
@@
 </segment>
 </net>
-<net name="N$3" class="0">
-<segment>
-<pinref part="U$16" gate="G$1" pin="P$1"/>
-<wire x1="-50.8" y1="40.64" x2="-58.42" y2="40.64" width="0.1524" layer="91"/>
-<pinref part="+3V12" gate="G$1" pin="+3V3"/>
-</segment>
-</net>
-<net name="N$6" class="0">
-<segment>
-<pinref part="U$17" gate="G$1" pin="P$1"/>
-<wire x1="-50.8" y1="27.94" x2="-55.88" y2="27.94" width="0.1524" layer="91"/>
-<pinref part="GND18" gate="1" pin="GND"/>
-</segment>
-</net>
